File: arrow_deca_retro_cape.kicad_sch (KiCad schematic)
At the start: 56 parts, among them J1 DB15_Female_HighDensity, J10 Conn_02x06_Odd_Even, J11 PMOD1, J12 PMOD2, J14 Conn_01x02, J15 Conn_01x03, J16 Conn_01x06, J17 Conn_01x02, J18 Conn_01x03, J19 DINC_MIN_TM_6_1, J20 PMOD3, J21 USB3_A, J22 Conn_01x03, J3 Conn_01x06, J4 DB9_Male_MountingHoles, J5 DINC_MIN_TM_6_1, J6 Conn_02x20_Odd_Even, J7 Conn_01x03, J8 P8_Male, J9 P9_Male, U4 LM1117-3.3, U5 LM1117-2.5

Commit message: v0.68 vga schematic
Parts:
- added R17, R18: 180, Resistor_SMD:R_0805_2012Metric_Pad1.20x1.40mm_HandSolder, symbol Device:R
- added R19, R20, R21, R25, R26, R27, R31, R32, R33: 2k, Resistor_SMD:R_0805_2012Metric_Pad1.20x1.40mm_HandSolder, symbol Device:R
- added R22, R23, R24, R28, R29, R30, R34, R35, R36: 1k, Resistor_SMD:R_0805_2012Metric_Pad1.20x1.40mm_HandSolder, symbol Device:R
- R1, R10, R11, R12, R13, R14, R15, R16, R2, R9: value 100 -> 180
- R5, R6: value 120 -> 180
Connections:
- net VGAB: now also R32.2, R33.2, R34.2, R35.2, R36.2
- net VGAG: now also R26.2, R27.2, R28.2, R29.2, R30.2
- net VGAR: now also R20.2, R21.2, R22.2, R23.2, R24.2
- net VGA_B0: now also R31.2
- net VGA_B1: now also R33.1
- net VGA_B2: now also R34.1
- net VGA_B3: now also R35.1, R36.1
- net VGA_G0: now also R25.2
- net VGA_G1: now also R27.1
- net VGA_G2: now also R28.1
- net VGA_G3: now also R29.1, R30.1
- net VGA_HS: now also R17.1
- net VGA_R0: now also R19.2
- net VGA_R1: now also R21.1
- net VGA_R2: now also R22.1
- net VGA_R3: now also R23.1, R24.1
- net VGA_VS: now also R18.1
- net VGA222_HS: no longer names the net of J1.13
- net VGA222_HS: now also R17.2
- net VGA222_VS: no longer names the net of J1.14
- net VGA222_VS: now also R18.2
- new net: R19.1, R20.1
- new net: R31.1, R32.1
- new net: R25.1, R26.1
Other:
- moved on the sheet: C18, C19, C20, C21, D1, D2, D3, D4, J1, J10, J14, J15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

Commit message: updated readme and routing improvement
Connections:
- net VGAHS: now reaches J1.13, R17.2
- net VGAVS: now reaches J1.14, R18.2
Other:
- moved on the sheet: D1, D10, D11, D12, D2, D5, D6, D7, D8, D9, J17, J20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

Commit message: update
Parts:
- removed J1: DB15_Female_HighDensity, vga:DSUB-15-HD_Female_Horizontal_P2.29x2.54mm_EdgePinOffset3.03mm_Housed_MountingHolesOffset4.94mm, symbol Connector:DB15_Female_HighDensity
- removed R7, R8: DNI, Resistor_SMD:R_0805_2012Metric_Pad1.20x1.40mm_HandSolder, symbol Device:R
- added J1: DB15_Female_HighDensity_MountingHoles, vga:DSUB-15-HD_Female_Horizontal_P2.29x2.54mm_EdgePinOffset3.03mm_Housed_MountingHolesOffset4.94mm, symbol Connector:DB15_Female_HighDensity_MountingHoles
- C18, C19: footprint Capacitor_SMD:C_0805_2012Metric_Pad1.15x1.40mm_HandSolder -> Capacitor_SMD:C_0805_2012Metric_Pad1.18x1.45mm_HandSolder
Connections:
- net GND: now also J1.0, J1.10, J1.5, J1.6, J1.7, J1.8
- net TX+: no longer J4.9
- net VGAB: now also J1.3
- net VGAG: now also J1.2
- net VGAHS: now also J1.13
- net VGAR: now also J1.1
- net VGAVS: now also J1.14
- net at D5.3, J22.1 (Pin_1), R9.2: now also J4.9
Other:
- note added: "-Buscar disponibilitat Condensadors"
- note added: "DETO PMOD (6 pin)"
- note removed: "-R2R VGA - REVISAR PINOUT, i2s retorn deca a DAC DETO 2, 3, 4 - I2S header al DETO PMOD"
- note removed: "DETO BUS (6 pin Pmod)"
- moved on the sheet: R17, R18, R19, R20, R21, R22, R23, R24, R25, R26, R27, R28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

Commit message: v0.71 gerbers sent for manufacturing
Parts:
- C18: value 10uF -> 1uF
- C19, C21: value 100uF -> 10uF
- C20: value 10uF -> 0.1uF
Changed lines of the file:
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@@
       (effects (font (size 1.27 1.27)) (justify left))
     )
-    (property "Value" "10uF" (id 1) (at 28.956 224.663 0)
+    (property "Value" "1uF" (id 1) (at 28.956 224.663 0)
       (effects (font (size 1.27 1.27)) (justify left))
     )
@@
       (effects (font (size 1.27 1.27)) (justify left))
     )
-    (property "Value" "100uF" (id 1) (at 51.816 224.663 0)
+    (property "Value" "10uF" (id 1) (at 51.816 224.663 0)
       (effects (font (size 1.27 1.27)) (justify left))
     )
@@
       (effects (font (size 1.27 1.27)) (justify left))
     )
-    (property "Value" "100uF" (id 1) (at 116.586 219.583 0)
+    (property "Value" "10uF" (id 1) (at 116.586 219.583 0)
       (effects (font (size 1.27 1.27)) (justify left))
     )
@@
       (effects (font (size 1.27 1.27)) (justify left))
     )
-    (property "Value" "10uF" (id 1) (at 96.266 219.583 0)
+    (property "Value" "0.1uF" (id 1) (at 96.266 219.583 0)
       (effects (font (size 1.27 1.27)) (justify left))
     )
@@
     )
     (path "/00000000-0000-0000-0000-0000612c6c71"
-      (reference "C18") (unit 1) (value "10uF") (footprint "Capacitor_SMD:C_0805_2012Metric_Pad1.18x1.45mm_HandSolder")
+      (reference "C18") (unit 1) (value "1uF") (footprint "Capacitor_SMD:C_0805_2012Metric_Pad1.18x1.45mm_HandSolder")
     )
     (path "/00000000-0000-0000-0000-000061573ffc"
-      (reference "C19") (unit 1) (value "100uF") (footprint "Capacitor_SMD:C_0805_2012Metric_Pad1.18x1.45mm_HandSolder")
+      (reference "C19") (unit 1) (value "10uF") (footprint "Capacitor_SMD:C_0805_2012Metric_Pad1.18x1.45mm_HandSolder")
     )
     (path "/dbc6bf33-0237-48dc-ae27-ad54518f632a"
-      (reference "C20") (unit 1) (value "10uF") (footprint "Capacitor_SMD:C_0805_2012Metric_Pad1.18x1.45mm_HandSolder")
+      (reference "C20") (unit 1) (value "0.1uF") (footprint "Capacitor_SMD:C_0805_2012Metric_Pad1.18x1.45mm_HandSolder")
     )
     (path "/b69a0113-a3fa-46ec-a4a8-820d383b62d2"
-      (reference "C21") (unit 1) (value "100uF") (footprint "Capacitor_SMD:C_0805_2012Metric_Pad1.18x1.45mm_HandSolder")
+      (reference "C21") (unit 1) (value "10uF") (footprint "Capacitor_SMD:C_0805_2012Metric_Pad1.18x1.45mm_HandSolder")
     )
     (path "/1c2f2557-8426-40eb-aec3-1be963f76a13"
