File: arrow_deca_retro_cape.kicad_sch (KiCad schematic)
At the start: 75 parts, among them J1 DB15_Female_HighDensity_Mount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, J10 Conn_02x06_Odd_Even, J11 PMOD1, J12 PMOD2, J14 Conn_01x02, J15 Conn_01x03, J16 Conn_01x06, J17 Conn_01x02, J18 Conn_01x03, J19 DINC_MIN_TM_6_1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

Commit message: v0.90 finalized gerger, bom and cpl files ready for jlcpcb production
Other:
- note added: "(**) Only USB3 or DB9 to be connected at the same time"
- note added: "2V5 GPIO"
- note added: "DB9 (**)"
- note added: "USB3 USER PORT (**)"
- note removed: "DB9"
- note removed: "Only USB3 or DB9 to be connected at the same time"
- note removed: "USB3 USER PORT"
- moved on the sheet: J10, J14, J21, JP7, JP8, JP9

Commit message: minor schematic notes update
Other:
- note removed: "(DI)"
- note removed: "(DO)"
Changed lines of the file:
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@@
     (effects (font (size 2 2)) (justify left bottom))
-  )
-  (text "(DI)" (at 200.66 97.155 0)
-    (effects (font (size 1.27 1.27)) (justify left bottom))
   )
   (text "(*)" (at 269.875 67.945 0)
@@
     (effects (font (size 2 2)) (justify left bottom))
   )
-  (text "(DO)" (at 200.66 94.615 0)
-    (effects (font (size 1.27 1.27)) (justify left bottom))
-  )
   (text "EXTERNAL MISTER MODULE" (at 336.55 21.59 0)
